File: Kicad/MCU.kicad_sch (KiCad schematic)
At the start: 24 parts, among them J201 Extension, J202 Debug, J203 Serial, J204 DCC, J205 Sense, U201 RaspberryPi_Pico2_Module-RP23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, U202 LM4040LP-3

Commit message: Centrale V2.3 (1)
Connections:
- net DCC-MON: no longer names the net of J204.3 (Pin_3)
- net DCC-MON: no longer U201.B7 (GPIO34)
- net LN-ENABLE: no longer names the net of U201.A38 (GPIO15)
- no-connect marks 6 -> 9
Changed lines of the file:
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@@
+	)
+	(no_connect
+		(at 127 86.36)
+	)
+	(no_connect
+		(at 274.32 92.71)
 	)
 	(no_connect
@@
 	(no_connect
 		(at 175.26 39.37)
+	)
+	(no_connect
+		(at 175.26 92.71)
 	)
 	(bus_entry
@@
 	(wire
 		(pts
-			(xy 121.92 86.36) (xy 127 86.36)
-		)
-		(stroke
-			(width 0)
-			(type default)
-		)
-	)
-	(wire
-		(pts
 			(xy 243.84 125.73) (xy 243.84 132.08)
 		)
@@
 	(wire
 		(pts
-			(xy 271.78 92.71) (xy 274.32 92.71)
-		)
-		(stroke
-			(width 0)
-			(type default)
-		)
-	)
-	(wire
-		(pts
 			(xy 121.92 104.14) (xy 127 104.14)
 		)
@@
 		(pts
 			(xy 127 109.22) (xy 36.83 109.22)
-		)
-		(stroke
-			(width 0)
-			(type default)
-		)
-	)
-	(wire
-		(pts
-			(xy 175.26 92.71) (xy 179.07 92.71)
 		)
 		(stroke
@@
 		)
 	)
-	(hierarchical_label "DCC-MON"
-		(shape input)
-		(at 179.07 92.71 0)
-		(effects
-			(font
-				(size 1.27 1.27)
-			)
-			(justify left)
-		)
-	)
 	(hierarchical_label "W5500-INT"
 		(shape input)
@@
 		)
 	)
-	(hierarchical_label "LN-ENABLE"
-		(shape output)
-		(at 121.92 86.36 180)
-		(effects
-			(font
-				(size 1.27 1.27)
-			)
-			(justify right)
-		)
-	)
 	(hierarchical_label "XpressNetTX"
 		(shape output)
@@
 		(effects
 			(font
-				(size 1.27 1.27)
-			)
-			(justify right)
-		)
-	)
-	(hierarchical_label "DCC-MON"
-		(shape input)
-		(at 271.78 92.71 180)
-		(effects
-			(font
