File: Kicad/TMC-Centrale-V2.2.kicad_pcb (KiCad board)
At the start: 2 copper layers, 180 x 90 mm, 129 parts, among them J1001 Loconet_Power, J1002 Loconet-T, J1003 LN_RX, J1004 LN_TX, J1005 LN_ACT, J1006 Loconet-B, J201 Extension, J202 Debug, J203 Serial, J204 DCC, J205 Sense, J301 GND, J302 GND, J303 Connector-Power-Barrel-Jack, J501 DIN-XpressNet, J502 XPN, J503 XpressNet, J601 DCC-OUT, J701 CDE, J801 DCC-SM, J901 RS-Bus, J902 RS_TX, J903 RS_RX, Q1001 BC547, Q1002 BC547, Q1003 BC547, Q901 BC557, Q902 IRLZ44N, Q903 BC547, U1001 LM393, U1002 UCC27425, U201 RaspberryPi_Pico2_Module-RP23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, U202 LM4040LP-3, U301 5V Step down Module, U302 12V Step down Module, U401 Module-W5500, U501 MAX3485, U601 DRV8874, U701 DRV8876, U801 DRV8874/8876

Commit message: Centrale V2.3 (1)
Parts:
- removed C1005: 100nF, Capacitor_THT:C_Disc_D5.0mm_W2.5mm_P2.50mm
- removed C1006, C1007: 4,7nF, Capacitor_THT:C_Rect_L10.0mm_W5.0mm_P5.00mm_P7.50mm
- removed DTVS1001, DTVS1002: P6KE15A, Diode_THT:D_DO-15_P12.70mm_Horizontal
- removed J1005: LN_ACT, Connector_PinHeader_2.54mm:PinHeader_1x01_P2.54mm_Vertical
- removed R1013, R1014: 33Ω (2W), Resistor_THT:R_Axial_DIN0516_L15.5mm_D5.0mm_P20.32mm_Horizontal
- removed U1002: UCC27425, AP_Library:DIL08
Connections:
- D701 pad 2: /CDE-Interface/C -> /CDE-Interface/DCC-C
- J1006 pad 1: /LocoNet/LN_OUTA -> /CDE-Interface/DCC-C
- J1006 pad 6: /LocoNet/LN_OUTB -> /CDE-Interface/DCC-D
- J204 pad 3: /LocoNet/DCC-MON -> unconnected-(J204-Pin_3-Pad3)
- J701 pad 1: /CDE-Interface/C -> /CDE-Interface/DCC-C
- J701 pad 2: /CDE-Interface/D -> /CDE-Interface/DCC-D
- U201 pad A38: /LocoNet/LN_ACTIVE -> unconnected-(U201-GPIO15-PadA38)
- U201 pad B7: /LocoNet/DCC-MON -> unconnected-(U201-GPIO34-PadB7)
- U701 pad 11: /CDE-Interface/D -> /CDE-Interface/DCC-D
- U701 pad 12: /CDE-Interface/C -> /CDE-Interface/DCC-C
Routing:
- net /LocoNet/DCC-MON: track 119.3 -> 0.00 mm, vias 2 -> 0
- net (no net): track 0.00 -> 74.5 mm, vias 0 -> 2
- net /LocoNet/LN_ACTIVE: track 72.8 -> 0.00 mm
- net GND: track 1188.5 -> 1118.8 mm, vias 17 -> 15
- net /CDE-Interface/DCC-C: track 0.00 -> 49.8 mm, vias 0 -> 1
- net /CDE-Interface/C: track 49.8 -> 0.00 mm, vias 1 -> 0
- net /LocoNet/LN_OUTB: track 45.2 -> 0.00 mm
- net /LocoNet/LN_OUTA: track 26.4 -> 0.00 mm
- net /CDE-Interface/DCC-D: track 0.00 -> 23.7 mm
- net /CDE-Interface/D: track 23.6 -> 0.00 mm
- net /12V: track 236.0 -> 215.8 mm
- net unconnected-(U201-GPIO15-PadA38): track 0.00 -> 17.4 mm
- net Net-(U1002-OUTB): track 4.59 -> 0.00 mm
- net Net-(U1002-OUTA): track 4.31 -> 0.00 mm
