File: Kicad/XpressNet.kicad_sch (KiCad schematic)
At the start: 10 parts, among them J501 DIN-XpressNet, J502 XPN, J503 XpressNet, U501 MAX3485

Commit message: Centrale V2.3 (1)
Changed lines of the file:
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@@
 	)
 	(hierarchical_label "XpressNetRX"
-		(shape input)
+		(shape output)
 		(at 250.19 67.31 180)
 		(effects
@@
 	)
 	(hierarchical_label "XpressNetRX"
-		(shape input)
+		(shape output)
 		(at 102.87 63.5 180)
 		(effects
